File: resetter.kicad_pcb (KiCad board)
At the start: 2 copper layers, 64.1 x 48.9 mm, 15 parts, among them J1 Conn_01x02_Female, J2 Conn_01x01, J3 Conn_01x02, J4 Conn_01x02, Q1 2N3904-AP, Q2 Q_PMOS_GDS, Q3 Q_PMOS_GDS, U1 VX7805, U2 adafruit_tpl5110

Commit message: update
Parts:
- removed MK1, MK2, MK3, MK4: Mounting_Hole, Mounting_Holes:MountingHole_2.2mm_M2_Pad
- moved U1 3.25 mm to (69.0, 33.9)
Routing:
- net Net-(U1-Pad3): track 10.2 -> 13.5 mm
- net Net-(J4-Pad2): track 46.5 -> 49.5 mm
- net GND: track 129.0 -> 130.1 mm
- net (no net): vias 0 -> 2
Other:
- board size 64.1 x 48.9 mm -> 54.7 x 43.3 mm
